File: ai03-modified.kicad_sch (KiCad schematic)
At the start: 20 parts, among them SW1 SW_Push, U1 ATmega32U4-A, Y1 16MHz

Commit message: Finish
Parts:
- USB1: footprint random-keyboard-parts:Molex-0548190589 -> random-keyboard-parts:Molex-0548190519
Connections:
- net ROW1 is gone; now on net ROW0: D2.1 (K)
- net GND: now also USB1.1 (GND), USB1.6 (SHIELD)
- net ROW0: now also U1.38 (PF5); no longer MX1.1 (COL), MX2.1 (COL)
- net VCC: now also USB1.5 (VBUS); no longer USB1.6 (SHIELD)
- net COL0: now reaches U1.37 (PF6)
- net COL0: now also MX1.1 (COL)
- net COL1: now reaches U1.40 (PF1)
- net COL1: now also MX2.1 (COL)
Other:
- moved on the sheet: D2, F1, MX2
